File: hardware/rev2/endeavour.kicad_pcb (KiCad board)
At the start: 2 copper layers, 82 x 54.2 mm, 75 parts, among them J1 UART, J2 HDMI_A, J3 USB_C_Receptacle_USB2.0, J4 SJ-2523-SMT-TR, J5 Micro_SD_Card_Det2, J6 USB_A, J7 USB_A, J8 Conn_01x04_Socket, J9 Conn_01x03_Socket, SW1 Push1, SW2 Push2, SW4 PB400EEQR1BLK, SW5 FTDI/DIRECT, SW6 SWx02, U1 10M50SAE144, U10 PAM8302AAD, U11 FT2232HL, U2 KC2520Z 100MHz, U3 AS4C64M16D1, U4 Si5351A-B-GT, U5 Si5351A-B-GT, U7 AP63203WU, U8 AP2114H-2.5TRG1, U9 MCP4726A0T-E/CH, Y1 12MHz, Y2 25MHz, Y3 25MHz

Commit message: rev2, clocks
Parts:
- removed C17: 10uF, Capacitor_SMD:C_0603_1608Metric
- removed C18: 0.1uF, Capacitor_SMD:C_0603_1608Metric
- removed R20, R21: 15K, Resistor_SMD:R_0603_1608Metric
- removed U10: PAM8302AAD, Package_SO:SOIC-8_3.9x4.9mm_P1.27mm
- added C13: 1uF, Capacitor_SMD:C_0603_1608Metric, B.Cu at (147.7, 81.5)
- added C14: 1uF, Capacitor_SMD:C_0603_1608Metric, B.Cu at (143.4, 76.5)
- added C15: 1uF, Capacitor_SMD:C_0603_1608Metric, B.Cu at (116.4, 91.2)
- added C5: 100uF, Capacitor_Tantalum_SMD:CP_EIA-3528-12_Kemet-T, B.Cu at (150.6, 72.1)
- added C6: 100uF, Capacitor_Tantalum_SMD:CP_EIA-3528-12_Kemet-T, B.Cu at (146.7, 72.1)
- added C7: 1uF, Capacitor_SMD:C_0603_1608Metric, B.Cu at (154.9, 70.5)
- added C8: 1uF, Capacitor_SMD:C_0603_1608Metric, B.Cu at (149.4, 81.5)
- added J10: Conn_02x05_Odd_Even, Connector_PinSocket_2.54mm:PinSocket_2x06_P2.54mm_Vertical, B.Cu at (103.9, 64.5)
- added J11: Conn_02x03_Odd_Even, Connector_PinSocket_2.54mm:PinSocket_2x03_P2.54mm_Vertical, B.Cu at (154.2, 64.5)
- added JP1: snd_power, Jumper:SolderJumper-3_P1.3mm_Open_Pad1.0x1.5mm, B.Cu at (143.2, 85.8)
- added R10: 560, Resistor_SMD:R_0603_1608Metric, B.Cu at (143.3, 94.0)
- added R11: 560, Resistor_SMD:R_0603_1608Metric, B.Cu at (143.3, 96.0)
- added REF**: MountingHole_2.2mm_M2, MountingHole:MountingHole_2.2mm_M2, F.Cu at (84.9, 63.2)
- added REF**: MountingHole_2.2mm_M2, MountingHole:MountingHole_2.2mm_M2, F.Cu at (160.4, 63.2)
- added U6: MCP4728, Package_SO:MSOP-10_3x3mm_P0.5mm, B.Cu at (148.3, 87.5)
- C12, C20: moved to F.Cu
- D1, D2, D3: footprint LED_THT:LED_D3.0mm -> LED_SMD:LED_0603_1608Metric
- D4: renamed from D8; footprint LED_THT:LED_D3.0mm -> LED_SMD:LED_0603_1608Metric
- J4: value SJ-2523-SMT-TR -> SJ-3523-SMT
- R1, R31: moved to B.Cu
- R4, R5, R6: value 1K -> 350; moved to B.Cu
- U9: value MCP4726A0T-E/CH -> LM4811; footprint Package_TO_SOT_SMD:SOT-23-6 -> Package_SO:TSSOP-10_3x3mm_P0.5mm
- moved U9 34.8 mm to (148.6, 77.5)
- moved C12 30.4 mm to (138.7, 114.5), turned to 90 degrees
- moved D3 26.8 mm to (119.2, 80.2), turned to 90 degrees
- moved R6 26.7 mm to (119.2, 80.3), turned to -90 degrees
- moved U8 25.9 mm to (139.1, 113.0), turned to 0 degrees
- moved C21 25.1 mm to (125.4, 83.0), turned to 90 degrees
- moved R5 25.1 mm to (116.7, 80.3), turned to -90 degrees
- moved D2 24.8 mm to (116.7, 80.2), turned to 90 degrees
- moved R4 23.0 mm to (114.2, 80.3), turned to -90 degrees
- moved D1 22.8 mm to (114.2, 80.2)
- moved C20 21.5 mm to (134.9, 115.2), turned to 0 degrees
- moved D4 21.0 mm to (84.4, 82.0)
- moved R1 19.0 mm to (123.4, 83.0), turned to -90 degrees
- moved R31 17.7 mm to (139.9, 63.1), turned to 90 degrees
- moved R16 16.5 mm to (95.7, 83.5)
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Connections:
- J4 pad 1: Net-(U10-OUT+) -> GND
- J4 pad 2: Net-(U10-OUT-) -> Net-(J11-Pin_6)
- J4 pad 3: Net-(U10-OUT-) -> Net-(J11-Pin_5)
- R16 pad 2: +5V -> +3.3V
- R6 pad 1: GND -> Net-(D3-A)
- R6 pad 2: Net-(D3-K) -> +2V5
- U1 pad 10: unconnected-(U1-io1A_10/ADC1IN4-Pad10) -> Net-(J10-Pin_8)
- U1 pad 100: unconnected-(U1-io6_100-Pad100) -> g100
- U1 pad 101: unconnected-(U1-io6_101-Pad101) -> g101
- U1 pad 102: unconnected-(U1-io6_102-Pad102) -> g102
- U1 pad 105: unconnected-(U1-io6_105-Pad105) -> TMDSCm
- U1 pad 106: unconnected-(U1-io6_106-Pad106) -> TMDSCp
- U1 pad 11: unconnected-(U1-io1A_11/ADC1IN5-Pad11) -> Net-(J10-Pin_7)
- U1 pad 110: unconnected-(U1-io7_110-Pad110) -> TMDS0m
- U1 pad 111: unconnected-(U1-io7_111-Pad111) -> TMDS0p
- U1 pad 116: unconnected-(U1-io7_116/VREFB7NO-Pad116) -> SND_SHDN
- U1 pad 117: unconnected-(U1-io7_117-Pad117) -> TMDS1m
- U1 pad 118: unconnected-(U1-io7_118-Pad118) -> TMDS1p
- U1 pad 119: unconnected-(U1-io7_119-Pad119) -> TMDS2m
- U1 pad 12: unconnected-(U1-io1A_12/ADC1IN6-Pad12) -> Net-(J10-Pin_10)
- U1 pad 120: unconnected-(U1-io7_120-Pad120) -> TMDS2p
- U1 pad 13: unconnected-(U1-io1A_13/ADC1IN7-Pad13) -> Net-(J10-Pin_9)
- U1 pad 134: Net-(D3-A) -> Net-(D3-K)
- U1 pad 14: unconnected-(U1-io1A_14/ADC1IN8-Pad14) -> Net-(J10-Pin_12)
- U1 pad 15: unconnected-(U1-io1B_15/JTAGEN-Pad15) -> Net-(J10-Pin_11)
- U1 pad 3: ANAIN_3 -> Net-(J10-Pin_4)
- U1 pad 6: unconnected-(U1-io1A_6/ADC1IN1-Pad6) -> Net-(J10-Pin_3)
- U1 pad 7: unconnected-(U1-io1A_7/ADC1IN2-Pad7) -> Net-(J10-Pin_6)
- U1 pad 8: unconnected-(U1-io1A_8/ADC1IN3-Pad8) -> Net-(J10-Pin_5)
- U1 pad 96: unconnected-(U1-io6_96/DPCLK3-Pad96) -> SND_SCL
- U1 pad 97: unconnected-(U1-io6_97/VREFB6N0-Pad97) -> SND_SDA
- U1 pad 98: unconnected-(U1-io6_98/DPCLK2-Pad98) -> USB_host2_Dm
- U1 pad 99: unconnected-(U1-io6_99-Pad99) -> USB_host2_Dp
- U3 pad 1: Net-(U3-VDD-Pad1) -> +2V5
- U3 pad 15: VDDQ -> +2V5
- U3 pad 18: Net-(U3-VDD-Pad1) -> +2V5
- U3 pad 3: VDDQ -> +2V5
- U3 pad 33: Net-(U3-VDD-Pad1) -> +2V5
- U3 pad 55: VDDQ -> +2V5
- U3 pad 61: VDDQ -> +2V5
- U3 pad 9: VDDQ -> +2V5
- U9 pad 2: GND -> Net-(U9-VIN1)
- U9 pad 3: +3.3V -> Net-(U9-BYPASS)
- U9 pad 4: SND_SDA -> Net-(U6-VOUTD)
- U9 pad 5: SND_SCL -> GND
- U9 pad 6: unconnected-(U9-A0-Pad6) -> Net-(U6-VOUTA)
Routing:
- net GND: track 457.3 -> 673.8 mm, vias 19 -> 33
- net +5V: track 40.6 -> 157.6 mm, vias 0 -> 1
- net +3.3V: track 204.8 -> 291.0 mm, vias 6 -> 9
- net Net-(J10-Pin_11): track 0.00 -> 52.8 mm
- net Net-(J10-Pin_10): track 0.00 -> 51.6 mm
- net Net-(J10-Pin_9): track 0.00 -> 49.3 mm
- net +2V5: track 98.7 -> 147.8 mm, vias 5 -> 8
- net Net-(J10-Pin_12): track 0.00 -> 47.6 mm
- net Net-(J10-Pin_7): track 0.00 -> 46.1 mm
- net Net-(J11-Pin_6): track 0.00 -> 45.3 mm, vias 0 -> 1
- net Net-(J10-Pin_5): track 0.00 -> 43.5 mm
- net Net-(J10-Pin_8): track 0.00 -> 42.5 mm
- net Net-(J10-Pin_3): track 0.00 -> 40.2 mm
- net Net-(J11-Pin_5): track 0.00 -> 39.9 mm, vias 0 -> 1
- net Net-(J10-Pin_6): track 0.00 -> 38.4 mm
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- added copper zone on B.Cu, net +3.3V
- added copper zone on B.Cu, net +5V
- added copper zone on B.Cu, net GND
- added copper zone on F.Cu, net GND
Other:
- board size 82 x 54.2 mm -> 82 x 58 mm
- board text added: "Endeavour rev 2"
- board text added: "SND L"
- board text added: "SND PWR"
- board text added: "SND R"
- board text added: "USB 1"
- board text added: "USB 2"
- board text added: "a10"
- board text added: "a11"
- board text added: "a12"
- board text added: "a13"
- board text added: "a14"
- board text added: "a6"
- board text added: "a7"
- board text added: "a8"
- board text added: "ai3"
- board text added: "g100"
- board text added: "g101"
- board text added: "g102"
- board text added: "g15"
