File: hardware/rev2/peripherals.kicad_sch (KiCad schematic)
At the start: 18 parts, among them J2 HDMI_A, J4 SJ-2523-SMT-TR, J5 Micro_SD_Card_Det2, J6 USB_A, J7 USB_A, U10 PAM8302AAD, U3 AS4C64M16D1, U9 MCP4726A0T-E/CH

Commit message: rev2, clocks
Parts:
- removed C17: 10uF, Capacitor_SMD:C_0603_1608Metric, symbol Device:C
- removed C18: 0.1uF, Capacitor_SMD:C_0603_1608Metric, symbol Device:C
- removed R17: PT01-D115D-B104, endeavour:TRIM_PT01-D115D-B104, symbol endeavour:PT01-D115D-B104
- removed R20, R21: 15K, Resistor_SMD:R_0603_1608Metric, symbol Device:R
- removed U10: PAM8302AAD, Package_SO:SOIC-8_3.9x4.9mm_P1.27mm, symbol Amplifier_Audio:PAM8302AAD
- removed U9: MCP4726A0T-E/CH, Package_TO_SOT_SMD:SOT-23-6, symbol Analog_DAC:MCP4725xxx-xCH
- added C13, C14, C7, C8: 1uF, Capacitor_SMD:C_0603_1608Metric, symbol Device:C
- added C5, C6: 100uF, Capacitor_Tantalum_SMD:CP_EIA-3528-12_Kemet-T, symbol Device:C
- added J11: Conn_02x03_Odd_Even, Connector_PinSocket_2.54mm:PinSocket_2x03_P2.54mm_Vertical, symbol Connector_Generic:Conn_02x03_Odd_Even
- added JP1: snd_power, Jumper:SolderJumper-3_P1.3mm_Open_Pad1.0x1.5mm, symbol Jumper:Jumper_3_Bridged12
- added R10, R11: 1K, Resistor_SMD:R_0603_1608Metric, symbol Device:R
- added U6: MCP4728, Package_SO:MSOP-10_3x3mm_P0.5mm, symbol Analog_DAC:MCP4728
- added U9: LM4811, Package_SO:TSSOP-10_3x3mm_P0.5mm, symbol Amplifier_Audio:LM4811
- J4: value SJ-2523-SMT-TR -> SJ-3523-SMT; symbol endeavour:SJ-2523-SMT-TR -> endeavour:SJ-3523-SMT
Connections:
- net VDDQ is gone; now on net +2V5: U3.15 (VDDQ), U3.3 (VDDQ), U3.55 (VDDQ), U3.61 (VDDQ), U3.9 (VDDQ)
- net +2V5: now also U3.1 (VDD), U3.14 (NC), U3.18 (VDD), U3.33 (VDD)
- net +3.3V: now also JP1.1 (A), R10.1, R11.1
- net +5V: now also JP1.3 (B)
- net GND: now also J4.1, C14.1, C7.2, J11.1 (Pin_1), U6.10 (VSS), U6.4 (~{LDAC}), U9.5 (GND)
- net SND_SCL: now also R11.2, U6.2 (SCL)
- net SND_SDA: now also R10.2, U6.3 (SDA)
- net at J4.3: now also C5.2, J11.5 (Pin_5); no longer J4.2
- new net: C14.2, JP1.2 (C), U6.1 (VDD), U9.10 (VDD)
- new net: C5.1, U9.1 (VOUT1)
- new net: C13.1, U6.7 (VOUTB)
- new net: C13.2, U9.8 (VIN2)
- new net: U6.6 (VOUTA), U9.6 (UP/DN)
- new net: C8.1, U6.8 (VOUTC)
- new net: U6.9 (VOUTD), U9.4 (CLOCK)
- new net: C7.1, U9.3 (BYPASS)
- new net: C8.2, U9.2 (VIN1)
- new net: C6.1, U9.9 (VOUT2)
- new net: C6.2, J11.6 (Pin_6), J4.2
- new net SND_SHDN: U9.7 (SHDN)
- new net g100: J11.2 (Pin_2)
- new net g101: J11.4 (Pin_4)
- new net g102: J11.3 (Pin_3)
- no-connect marks 10 -> 9
Other:
- moved on the sheet: J4
