File: hardware/rev2/endeavour.kicad_sch (KiCad schematic)
At the start: 15 parts, among them SW1 Push1, SW2 Push2, U1 10M50SAE144, U2 KC2520Z 100MHz, U4 Si5351A-B-GT, U5 Si5351A-B-GT, Y2 25MHz, Y3 25MHz

Commit message: rev2, clocks
Parts:
- added J10: Conn_02x06_Odd_Even, Connector_PinSocket_2.54mm:PinSocket_2x06_P2.54mm_Vertical, symbol Connector_Generic:Conn_02x06_Odd_Even
- D1, D2, D3: footprint LED_THT:LED_D3.0mm -> LED_SMD:LED_0603_1608Metric
- R4, R5, R6: value 1K -> 350
Connections:
- net +2V5: now also R6.2
- net +3.3V: now also J10.2 (Pin_2)
- net GND: now also J10.1 (Pin_1); no longer R6.1
- net at D3.1 (K): now also U1.134 (io8_134/CRC_ERROR); no longer R6.2
- net at D3.2 (A): now also R6.1; no longer U1.134 (io8_134/CRC_ERROR)
- net at U1.10 (io1A_10/ADC1IN4): now also J10.8 (Pin_8)
- net g100: now reaches U1.100 (io6_100)
- net g101: now reaches U1.101 (io6_101)
- net g102: now reaches U1.102 (io6_102)
- net TMDSCm: now reaches U1.105 (io6_105)
- net TMDSCp: now reaches U1.106 (io6_106)
- net at U1.11 (io1A_11/ADC1IN5): now also J10.7 (Pin_7)
- net TMDS0m: now reaches U1.110 (io7_110)
- net TMDS0p: now reaches U1.111 (io7_111)
- net SND_SHDN: now reaches U1.116 (io7_116/VREFB7NO)
- net TMDS1m: now reaches U1.117 (io7_117)
- net TMDS1p: now reaches U1.118 (io7_118)
- net TMDS2m: now reaches U1.119 (io7_119)
- net at U1.12 (io1A_12/ADC1IN6): now also J10.10 (Pin_10)
- net TMDS2p: now reaches U1.120 (io7_120)
- net at U1.13 (io1A_13/ADC1IN7): now also J10.9 (Pin_9)
- net at U1.14 (io1A_14/ADC1IN8): now also J10.12 (Pin_12)
- net at U1.15 (io1B_15/JTAGEN): now also J10.11 (Pin_11)
- net at U1.6 (io1A_6/ADC1IN1): now also J10.3 (Pin_3)
- net at U1.7 (io1A_7/ADC1IN2): now also J10.6 (Pin_6)
- net at U1.8 (io1A_8/ADC1IN3): now also J10.5 (Pin_5)
- net SND_SCL: now reaches U1.96 (io6_96/DPCLK3)
- net SND_SDA: now reaches U1.97 (io6_97/VREFB6N0)
- net USB_host2_Dm: now reaches U1.98 (io6_98/DPCLK2)
- net USB_host2_Dp: now reaches U1.99 (io6_99)
- net ANAIN_3: no longer names the net of U1.3 (ANAIN1_3)
- net ANAIN_3: now also J10.4 (Pin_4)
Other:
- moved on the sheet: D3, R6

Commit message: update
Parts:
- R4, R5, R6: value 350 -> 300
Changed lines of the file:
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@@
       (effects (font (size 1.27 1.27)))
     )
-    (property "Value" "350" (at 256.54 45.72 90)
+    (property "Value" "300" (at 256.54 45.72 90)
       (effects (font (size 1.27 1.27)))
     )
@@
       (effects (font (size 1.27 1.27)))
     )
-    (property "Value" "350" (at 255.27 35.56 90)
+    (property "Value" "300" (at 255.27 35.56 90)
       (effects (font (size 1.27 1.27)))
     )
@@
       (effects (font (size 1.27 1.27)))
     )
-    (property "Value" "350" (at 256.54 55.88 90)
-      (effects (font (size 1.27 1.27)))
-    )
+    (property "Value" "300" (at 256.54 55.88 90)
+      (effects (font (size 1.27 1.27)))
+    )
